File: KiCad Files/Bojen_PCB/Bojen_PCB.kicad_pcb (KiCad board)
At the start: 2 copper layers, 195 x 88 mm, 41 parts, among them J1 5V Power In, J10 GPS EN, J2 Battery Voltage, J20 TMP PUL UP, J21 TMP PULL DOWN, J22 TMP Sens, J24 TDS Sens, J25 PH Sens, J26 DO Sens, J27 TRB Sens, J3 GPIO Breakout 2, J4 5V TFT, J5 3.3V TFT, J6 LED, J8 GPIO Breakout 1, J9 PWR TMR SKIP, Q1 IRF5210PBF, U1 Display_TFT_1.8Zoll_ST7735, U11 DO Sensor, U13 Solar Controller, U15 PH Sensor, U2 NEO-GPS8M, U3 SIM800L-CORE, U4 TLP5110 Power Timer Modul, U5 ADC - ADS1115 Module, U6 PCF8575 Module, U7 ESP32-DEVKIT-V1, U8 TDS Sensor, U9 Turbidity Sensor

Commit message: tft Screen QR Code Display
Other:
- board text added: "- D +"
- board text removed: "- + D"
Changed lines of the file:
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@@
 		)
 	)
-	(gr_text "-  +  D"
-		(at 210.185 102.235 90)
+	(gr_text "-  D  +"
+		(at 209.55 101.6 90)
 		(layer "F.SilkS")
 		(effects

Commit message: PCB Updated, Fixes
Parts:
- added C1: 100u, Capacitor_THT:CP_Radial_D8.0mm_P5.00mm, B.Cu at (41.6, 112.5)
- added C10: ?, Capacitor_THT:C_Axial_L5.1mm_D3.1mm_P10.00mm_Horizontal, F.Cu at (84.5, 106.5)
- added C11: 100u, Capacitor_THT:CP_Radial_D8.0mm_P5.00mm, B.Cu at (138.9, 100.0)
- added C12: 10u, Capacitor_THT:C_Axial_L5.1mm_D3.1mm_P10.00mm_Horizontal, F.Cu at (164.0, 92.5)
- added C13: 1u, Capacitor_THT:C_Axial_L5.1mm_D3.1mm_P10.00mm_Horizontal, F.Cu at (174.5, 106.0)
- added C2: 10u, Capacitor_THT:C_Axial_L5.1mm_D3.1mm_P10.00mm_Horizontal, F.Cu at (107.5, 102.5)
- added C3: 100u, Capacitor_THT:CP_Radial_D8.0mm_P5.00mm, B.Cu at (139.4, 120.0)
- added C4: 10u, Capacitor_THT:C_Axial_L5.1mm_D3.1mm_P10.00mm_Horizontal, B.Cu at (70.5, 115.5)
- added C5: 100u, Capacitor_THT:CP_Radial_D8.0mm_P5.00mm, B.Cu at (139.4, 79.0)
- added C6: 10u, Capacitor_THT:C_Axial_L5.1mm_D3.1mm_P10.00mm_Horizontal, F.Cu at (183.0, 99.5)
- added C6: 10u, Capacitor_THT:C_Axial_L5.1mm_D3.1mm_P10.00mm_Horizontal, F.Cu at (174.5, 112.0)
- added C7: 1u, Capacitor_THT:C_Axial_L5.1mm_D3.1mm_P10.00mm_Horizontal, F.Cu at (164.0, 86.5)
- added C8: ?, Capacitor_THT:C_Axial_L5.1mm_D3.1mm_P10.00mm_Horizontal, F.Cu at (84.5, 90.5)
- added C9: 1u, Capacitor_THT:C_Axial_L5.1mm_D3.1mm_P10.00mm_Horizontal, F.Cu at (107.5, 95.0)
- added J23: TMP PULL UP / DOWN, Connector_PinHeader_2.54mm:PinHeader_1x03_P2.54mm_Vertical, F.Cu at (198.5, 97.1)
- added J29: Sim PWR Skip, Connector_PinHeader_2.54mm:PinHeader_1x02_P2.54mm_Vertical, B.Cu at (43.5, 122.0)
- J20: value TMP PUL UP -> PCF_GPIO1; footprint Connector_PinHeader_2.54mm:PinHeader_1x02_P2.54mm_Vertical -> Connector_PinHeader_2.54mm:PinHeader_2x08_P2.54mm_Vertical; moved to B.Cu
- J21: value TMP PULL DOWN -> PCF_GPIO2; footprint Connector_PinHeader_2.54mm:PinHeader_1x02_P2.54mm_Vertical -> Connector_PinHeader_2.54mm:PinHeader_2x08_P2.54mm_Vertical; moved to B.Cu
- J24, J27: moved to B.Cu
- moved J20 55.9 mm to (177.6, 134.5), turned to 90 degrees
- moved J21 50.4 mm to (179.0, 66.0), turned to 90 degrees
- moved J10 25.3 mm to (184.8, 108.0), turned to 90 degrees
- moved J8 16.4 mm to (112.8, 69.4)
- moved J3 14.5 mm to (115.3, 127.2)
- moved J25 11.3 mm to (126.0, 81.0)
- moved J26 11.2 mm to (126.0, 122.0)
- moved U7 8.44 mm to (123.0, 99.0)
- moved R6 6.62 mm to (206.0, 91.1), turned to 180 degrees
- moved R5 4.61 mm to (198.2, 108.6), turned to 0 degrees
- moved J22 3.94 mm to (205.7, 102.0)
- moved J24 0.98 mm to (34.0, 118.0)
- moved J27 0.98 mm to (34.0, 84.4)
Connections:
- J20 pad 1: Net-(J20-Pin_1) -> /P00
- J20 pad 2: /TMP_SENS -> unconnected-(J20-Pin_2-Pad2)
- J21 pad 1: /TMP_SENS -> /P10
- J21 pad 2: Net-(J21-Pin_2) -> /ADC_ALRT
- R5 pad 1: Net-(J21-Pin_2) -> Net-(J23-Pin_3)
- R6 pad 2: Net-(J20-Pin_1) -> Net-(J23-Pin_1)
- U3 pad 3: unconnected-(U3-RST-Pad3) -> /SIM_RST
- U6 pad 1: /ADC_ALRT -> /P10
- U6 pad 13: unconnected-(U6-P00-Pad13) -> /P00
- U6 pad 14: unconnected-(U6-P01-Pad14) -> /P01
- U6 pad 15: unconnected-(U6-P02-Pad15) -> /P02
- U6 pad 16: unconnected-(U6-P03-Pad16) -> /P03
- U6 pad 17: unconnected-(U6-P04-Pad17) -> /P04
- U6 pad 18: unconnected-(U6-P05-Pad18) -> /P05
- U6 pad 19: /~SIM_EN -> /P06
- U6 pad 2: unconnected-(U6-P11-Pad2) -> /P11
- U6 pad 20: /SIM_DTR -> /P07
- U6 pad 3: unconnected-(U6-P12-Pad3) -> /P12
- U6 pad 4: unconnected-(U6-P13-Pad4) -> /P13
- U6 pad 5: unconnected-(U6-P14-Pad5) -> /P14
- U6 pad 6: unconnected-(U6-P15-Pad6) -> /P15
- U6 pad 7: unconnected-(U6-P16-Pad7) -> /P16
- U6 pad 8: unconnected-(U6-P17-Pad8) -> /P17
Routing:
- net /~SIM_EN: track 235.7 -> 0.00 mm, vias 1 -> 0
- net /sensors/ADC3: track 213.6 -> 0.00 mm, vias 1 -> 0
- net /SIM_DTR: track 209.4 -> 0.00 mm, vias 2 -> 0
- net /sensors/ADC0: track 186.5 -> 0.00 mm
- net /I2C_SDA: track 153.2 -> 0.00 mm, vias 2 -> 0
- net /I2C_SCL: track 145.4 -> 0.00 mm, vias 2 -> 0
- net /RX1: track 133.9 -> 0.00 mm, vias 1 -> 0
- net /TX1: track 125.8 -> 0.00 mm, vias 1 -> 0
- net /TMP_SENS: track 124.4 -> 0.00 mm, vias 1 -> 0
- net /TFT_CS: track 104.3 -> 0.00 mm, vias 2 -> 0
- net /TFT_DC: track 102.2 -> 0.00 mm, vias 1 -> 0
- net /sensors/ADC1: track 97.5 -> 0.00 mm, vias 1 -> 0
- net /SPI_SCK: track 96.9 -> 0.00 mm, vias 2 -> 0
- net /TFT_RST: track 96.7 -> 0.00 mm, vias 2 -> 0
- net /SPI_MISO: track 88.4 -> 0.00 mm, vias 1 -> 0
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Other:
- board text added: "ADC ALRT"
- board text added: "D12"
- board text added: "D13"
- board text added: "D14"
- board text added: "D15"
- board text added: "D16"
- board text added: "D17"
- board text added: "D18"
- board text added: "D19"
- board text added: "D2 led"
- board text added: "D21"
- board text added: "D22"
- board text added: "D23"
- board text added: "D25"
- board text added: "D26"
- board text added: "D27"
- board text added: "D32"
- board text added: "D33"
- board text added: "D34"
- board text added: "D35"
- board text added: "D4"
- board text added: "D5"
- board text added: "DOWN"
- board text added: "I2C_SCL"
- board text added: "I2C_SDA"
- board text added: "P00"
- board text added: "P01"
- board text added: "P02"
- board text added: "P03"
- board text added: "P04"
- board text added: "P05"
- board text added: "P06"
- board text added: "P07"
- board text added: "P10"
- board text added: "P11"
- board text added: "P12"
- board text added: "P13"
- board text added: "P14"
- board text added: "P15"
- board text added: "P16"
- board text added: "P17"
- board text added: "PULL UP"
- board text added: "PWR_DONE"
- board text added: "RX0"
- board text added: "RX1_GPS"
- board text added: "RX2_SIM"
- board text added: "SD_CS"
- board text added: "SIM DTR"
- board text added: "SIM RST"
- board text added: "SPI_MISO"
- board text added: "SPI_MOSI"
- board text added: "SPI_SCK"
- board text added: "TFT_CS"
- board text added: "TFT_DC"
- board text added: "TFT_RST"
- board text added: "TMP_SNS"
- board text added: "TX0"
- board text added: "TX1_GPS"
- board text added: "TX2_SIM"
- board text added: "VN"
- board text added: "VP"
- board text added: "X"
- board text added: "~SIM EN"
- board text removed: "Pull Down"
- board text removed: "Pull Up"
