File: KiCad Files/Bojen_PCB/sensors.kicad_sch (KiCad schematic)
At the start: 14 parts, among them J20 TMP PUL UP, J21 TMP PULL DOWN, J22 TMP Sens, J24 TDS Sens, J25 PH Sens, J26 DO Sens, J27 TRB Sens, U11 DO Sensor, U15 PH Sensor, U5 ADC - ADS1115 Module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

Commit message: PCB Updated, Fixes
Parts:
- removed J20: TMP PUL UP, Connector_PinHeader_2.54mm:PinHeader_1x02_P2.54mm_Vertical, symbol Connector_Generic:Conn_01x02
- removed J21: TMP PULL DOWN, Connector_PinHeader_2.54mm:PinHeader_1x02_P2.54mm_Vertical, symbol Connector_Generic:Conn_01x02
- added J23: TMP PULL UP / DOWN, Connector_PinHeader_2.54mm:PinHeader_1x03_P2.54mm_Vertical, symbol Connector_Generic:Conn_01x03
Connections:
- net TMP_Sens: now also J23.2 (Pin_2)
- net at R5.1: now also J23.3 (Pin_3)
- net at R6.2: now also J23.1 (Pin_1)
Changed lines of the file:
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@@
 	(wire
 		(pts
-			(xy 189.23 95.25) (xy 176.53 95.25)
+			(xy 176.53 95.25) (xy 189.23 95.25)
+		)
+		(stroke
+			(width 0)
+			(type default)
+		)
+	)
+	(wire
+		(pts
+			(xy 189.23 90.17) (xy 189.23 92.71)
 		)
 		(stroke
@@
 	(wire
 		(pts
-			(xy 189.23 92.71) (xy 189.23 95.25)
+			(xy 189.23 95.25) (xy 201.93 95.25)
 		)
 		(stroke
@@
 	(wire
 		(pts
+			(xy 189.23 97.79) (xy 189.23 100.33)
+		)
+		(stroke
+			(width 0)
+			(type default)
+		)
+	)
+	(wire
+		(pts
 			(xy 189.23 107.95) (xy 186.69 107.95)
 		)
@@
 	(wire
 		(pts
-			(xy 189.23 95.25) (xy 189.23 97.79)
-		)
-		(stroke
-			(width 0)
-			(type default)
-		)
-	)
-	(wire
-		(pts
 			(xy 167.64 49.53) (xy 173.99 49.53)
 		)
@@
 		(pts
 			(xy 186.69 82.55) (xy 189.23 82.55)
-		)
-		(stroke
-			(width 0)
-			(type default)
-		)
-	)
-	(wire
-		(pts
-			(xy 189.23 95.25) (xy 201.93 95.25)
 		)
 		(stroke
@@
 	)
 	(symbol
-		(lib_id "Connector_Generic:Conn_01x02")
-		(at 194.31 97.79 0)
-		(unit 1)
-		(exclude_from_sim no)
-		(in_bom yes)
-		(on_board yes)
-		(dnp no)
-		(property "Reference" "J21"
-			(at 196.85 97.536 90)
-			(effects
-				(font
-					(size 1.27 1.27)
-				)
-				(justify right)
-			)
-		)
-		(property "Value" "TMP PULL DOWN"
-			(at 211.836 103.124 0)
-			(effects
-				(font
-					(size 1.27 1.27)
-				)
-				(justify right)
-			)
-		)
-		(property "Footprint" "Connector_PinHeader_2.54mm:PinHeader_1x02_P2.54mm_Vertical"
-			(at 194.31 97.79 0)
+		(lib_id "Connector_Generic:Conn_01x03")
+		(at 194.31 95.25 0)
+		(unit 1)
+		(exclude_from_sim no)
+		(in_bom yes)
+		(on_board yes)
+		(dnp no)
+		(property "Reference" "J23"
+			(at 196.596 92.964 0)
+			(effects
+				(font
+					(size 1.27 1.27)
+				)
+				(justify left)
+			)
+		)
+		(property "Value" "TMP PULL UP / DOWN"
+			(at 196.088 98.298 0)
+			(effects
+				(font
+					(size 1.27 1.27)
+				)
+				(justify left)
+			)
+		)
+		(property "Footprint" "Connector_PinHeader_2.54mm:PinHeader_1x03_P2.54mm_Vertical"
+			(at 194.31 95.25 0)
 			(effects
 				(font
@@
 		)
 		(property "Datasheet" "~"
-			(at 194.31 97.79 0)
-			(effects
-				(font
-					(size 1.27 1.27)
-				)
-				(hide yes)
-			)
-		)
-		(property "Description" "Generic connector, single row, 01x02, script generated (kicad-library-utils/schlib/autogen/connector/)"
-			(at 194.31 97.79 0)
+			(at 194.31 95.25 0)
+			(effects
+				(font
+					(size 1.27 1.27)
+				)
+				(hide yes)
+			)
+		)
+		(property "Description" "Generic connector, single row, 01x03, script generated (kicad-library-utils/schlib/autogen/connector/)"
+			(at 194.31 95.25 0)
 			(effects
 				(font
@@
 		(pin "1"
 		)
+		(pin "3"
+		)
 		(pin "2"
 		)
 		(instances
-			(project "Bojen_PCB"
-				(path "/88bb7a71-704b-4bd6-bab4-d44bdefe0db1/18258186-5d10-4a41-839d-bac5b0a5fb0d"
-					(reference "J21")
+			(project ""
+				(path "/88bb7a71-704b-4bd6-bab4-d44bdefe0db1/18258186-5d10-4a41-839d-bac5b0a5fb0d"
+					(reference "J23")
 					(unit 1)
 				)
@@
 					(unit 1)
 				)
-			)
-		)
-	)
-	(symbol
-		(lib_id "Connector_Generic:Conn_01x02")
-		(at 194.31 90.17 0)
-		(unit 1)
-		(exclude_from_sim no)
-		(in_bom yes)
-		(on_board yes)
-		(dnp no)
-		(property "Reference" "J20"
-			(at 196.85 89.916 90)
-			(effects
-				(font
-					(size 1.27 1.27)
-				)
-				(justify right)
-			)
-		)
-		(property "Value" "TMP PUL UP"
-			(at 209.804 88.9 0)
-			(effects
-				(font
-					(size 1.27 1.27)
-				)
-				(justify right)
-			)
-		)
-		(property "Footprint" "Connector_PinHeader_2.54mm:PinHeader_1x02_P2.54mm_Vertical"
-			(at 194.31 90.17 0)
-			(effects
-				(font
-					(size 1.27 1.27)
-				)
-				(hide yes)
-			)
-		)
-		(property "Datasheet" "~"
-			(at 194.31 90.17 0)
-			(effects
-				(font
-					(size 1.27 1.27)
-				)
-				(hide yes)
-			)
-		)
-		(property "Description" "Generic connector, single row, 01x02, script generated (kicad-library-utils/schlib/autogen/connector/)"
-			(at 194.31 90.17 0)
-			(effects
-				(font
-					(size 1.27 1.27)
-				)
-				(hide yes)
-			)
-		)
-		(pin "1"
-		)
-		(pin "2"
-		)
-		(instances
-			(project "Bojen_PCB"
-				(path "/88bb7a71-704b-4bd6-bab4-d44bdefe0db1/18258186-5d10-4a41-839d-bac5b0a5fb0d"
-					(reference "J20")
-					(unit 1)
-				)
