File: KiCad Files/Bojen_PCB/Bojen_PCB.kicad_sch (KiCad schematic)
At the start: 9 parts, among them J1 5V Power In, J2 Battery Voltage, U1 Display_TFT_1.8Zoll_ST7735, U2 NEO-GPS8M, U3 SIM800L-CORE, U4 TLP5110 Adafruit Modul, U5 ADS1115 Module, U6 PCF8575 Module, U7 ESP32-DEVKIT-V1

Commit message: PCB Design
Parts:
- removed U3: SIM800L-CORE, Datenbojen:SIM800L-CORE, symbol alexandros444_lib:SIM800L-CORE
- removed U5: ADS1115 Module, Datenbojen:ADS1115 Module, symbol alexandros444_lib:ADS1115 Module
- removed U7: ESP32-DEVKIT-V1, Datenbojen:MODULE_ESP32_DEVKIT_V1, symbol ESP_Wroom_Dev:ESP32-DEVKIT-V1
- added J10: GPS EN, Connector_PinHeader_2.54mm:PinHeader_1x02_P2.54mm_Vertical, symbol Connector_Generic:Conn_01x02
- added J11, J12, J13, J14, J15, J16, J17, J18, J19, J7: Conn_02x08_Odd_Even, Connector_PinHeader_2.54mm:PinHeader_2x08_P2.54mm_Vertical, symbol Connector_Generic:Conn_02x08_Odd_Even
- added J4: 5V TFT, Connector_PinHeader_2.54mm:PinHeader_1x02_P2.54mm_Vertical, symbol Connector_Generic:Conn_01x02
- added J5: 3.3V TFT, Connector_PinHeader_2.54mm:PinHeader_1x02_P2.54mm_Vertical, symbol Connector_Generic:Conn_01x02
- added J6: LED, Connector_JST:JST_XH_B3B-XH-A_1x03_P2.50mm_Vertical, symbol Connector:Conn_01x03_Socket
- added J9: PWR TMR SKIP, Connector_PinHeader_2.54mm:PinHeader_1x02_P2.54mm_Vertical, symbol Connector_Generic:Conn_01x02
- added R3: 220k, Resistor_THT:R_Axial_DIN0207_L6.3mm_D2.5mm_P7.62mm_Horizontal, symbol Device:R
- added R4: 330, Resistor_THT:R_Axial_DIN0207_L6.3mm_D2.5mm_P7.62mm_Horizontal, symbol Device:R
- added U10: PH Sensor, Datenbojen:PH Sensor DFRobot, symbol alexandros444_lib:Sensor_DFRobot
- added U11: DO Sensor, Datenbojen:DO Sensor DFRobot, symbol alexandros444_lib:Sensor_DFRobot
- added U12: TMP Sensor, Datenbojen:Tempterature Sensor DFRobot, symbol alexandros444_lib:Sensor_DFRobot
- added U5: ADC - ADS1115 Module, Datenbojen:ADC - ADS1115 Module no hole, symbol alexandros444_lib:ADC - ADS1115 Module
- added U8: TDS Sensor, Datenbojen:TDS Sensor DFRobot, symbol alexandros444_lib:Sensor_DFRobot
- added U9: Turbidity Sensor, Datenbojen:Turbidity Sensor DFRobot, symbol alexandros444_lib:Sensor_DFRobot
- U1: footprint Datenbojen:ST7735 TFT Screen 1.8 Zoll -> Datenbojen:ST7735 TFT Screen 1.8 Zoll no hole
- U2: footprint Datenbojen:GY-NEO8MV2 -> Datenbojen:GY-NEO8MV2 no hole
- U4: value TLP5110 Adafruit Modul -> TLP5110 Power Timer Modul; footprint Datenbojen:TPL5110 Board -> Datenbojen:TPL5110 Board no hole
Connections:
- net GND: now also J2.1 (Pin_1), U1.7 (GND), U2.2 (GND), U6.10 (GND), U6.11 (GND), U6.C1 (GND), J6.1 (Pin_1), R3.2, U10.1 (GND), U11.1 (GND), U12.1 (GND), U5.2 (GND), U8.1 (GND), U9.1 (GND)
- net at U1.1 (TFT_LED): now also J5.1 (Pin_1)
- net SPI_MOSI: now reaches U1.10 (SD_MOSI)
- net SPI_MOSI: now also U1.3 (TFT_SDA_MOSI)
- net SPI_MISO: now reaches U1.11 (SD_MISO)
- net SPI_SCK: now reaches U1.12 (SD_SCK)
- net SPI_SCK: now also U1.2 (TFT_SCK)
- net TFT_DC: now reaches U1.4 (TFT_A0_DC)
- net TFT_RST: now reaches U1.5 (TFT_RST)
- net TFT_CS: now reaches U1.6 (TFT_CS)
- net at U1.8 (VCC): now also J4.2 (Pin_2)
- net SD_CS: now reaches U1.9 (SD_CS)
- net ADC_ALRT: now reaches U6.1 (P10)
- net ADC_ALRT: now also U5.6 (ALRT)
- net +5V: now reaches U6.12 (VDD)
- net +5V: now also U4.4 (DRV), U6.9 (VDD), U6.C2 (VCC), J10.2 (Pin_2), J4.1 (Pin_1), J6.3 (Pin_3), J9.2 (Pin_2), U10.2 (VCC), U11.2 (VCC), U12.2 (VCC), U5.1 (VCC), U8.2 (VCC), U9.2 (VCC)
- net ~SIM_EN: now reaches U6.19 (P06)
- net SIM_DTR: now reaches U6.20 (P07)
- net I2C_SDA: now reaches U6.C3 (SDA)
- net I2C_SDA: now also U5.4 (SDA)
- net I2C_SCL: now reaches U6.C4 (SCL)
- net I2C_SCL: now also U5.3 (SCL)
- net at J1.2 (Pin_2), U4.1 (VDD): now also J9.1 (Pin_1)
- net at U2.1 (VCC): now also J10.1 (Pin_1)
- net RX1: now reaches U2.3 (TX)
- net TX1: now reaches U2.4 (RX)
- net +BATT: now reaches J2.2 (Pin_2)
- net at U4.3 (Delay): now also R3.1
- net PWR_Done: now reaches U4.5 (Done)
- new net: J6.2 (Pin_2), R4.1
- new net +3.3V: J5.2 (Pin_2)
- new net ADC0: U5.7 (A0), U8.3 (A)
- new net ADC1: U5.8 (A1), U9.3 (A)
- new net ADC2: U10.3 (A), U5.9 (A2)
- new net ADC3: U11.3 (A), U5.10 (A3)
- new net LED_D: R4.2
- new net TMP_SENS: U12.3 (A)
- no-connect marks 7 -> 178
Other:
- added sheet ESP32 (ESP32.kicad_sch)
- added sheet SIM800L (SIM800L.kicad_sch)
- note added: "Eigentlich D weil Digital"
- moved on the sheet: J1, J2, U1, U2, U4, U6

Commit message: PCB V2
Parts:
- removed U10: PH Sensor, Datenbojen:PH Sensor DFRobot, symbol alexandros444_lib:Sensor_DFRobot
- removed U11: DO Sensor, Datenbojen:DO Sensor DFRobot, symbol alexandros444_lib:Sensor_DFRobot
- removed U12: TMP Sensor, Datenbojen:Tempterature Sensor DFRobot, symbol alexandros444_lib:Sensor_DFRobot
- removed U5: ADC - ADS1115 Module, Datenbojen:ADC - ADS1115 Module no hole, symbol alexandros444_lib:ADC - ADS1115 Module
- removed U8: TDS Sensor, Datenbojen:TDS Sensor DFRobot, symbol alexandros444_lib:Sensor_DFRobot
- removed U9: Turbidity Sensor, Datenbojen:Turbidity Sensor DFRobot, symbol alexandros444_lib:Sensor_DFRobot
- added H1, H2, H3, H4: MountingHole, MountingHole:MountingHole_3.2mm_M3, symbol Mechanical:MountingHole
- added U13: Solar Controller, Datenbojen:Solar Power MPPT Module, symbol alexandros444_lib:Solar_Controller
Connections:
- no-connect marks 178 -> 177
Other:
- added sheet sensors (sensors.kicad_sch)
- note removed: "Eigentlich D weil Digital"
- moved on the sheet: J6, R4

Commit message: PCB Updated, Fixes
Parts:
- added C1, C11, C5: 100u, Capacitor_THT:CP_Radial_D8.0mm_P5.00mm, symbol Device:C_Polarized
- added C10, C8: ?, Capacitor_THT:C_Axial_L5.1mm_D3.1mm_P10.00mm_Horizontal, symbol Device:C
- added C12, C2, C6: 10u, Capacitor_THT:C_Axial_L5.1mm_D3.1mm_P10.00mm_Horizontal, symbol Device:C
- added C13, C7, C9: 1u, Capacitor_THT:C_Axial_L5.1mm_D3.1mm_P10.00mm_Horizontal, symbol Device:C
- added J20: PCF_GPIO1, Connector_PinHeader_2.54mm:PinHeader_2x08_P2.54mm_Vertical, symbol Connector_Generic:Conn_02x08_Odd_Even
- added J21: PCF_GPIO2, Connector_PinHeader_2.54mm:PinHeader_2x08_P2.54mm_Vertical, symbol Connector_Generic:Conn_02x08_Odd_Even
- added J28: USB_A, Connector_USB:USB_A_Connfly_DS1095, symbol Connector:USB_A
Connections:
- net +3.3V: now also C11.1, C12.1, C13.1
- net +5V: now also C1.1, C10.1, C2.1, C5.1, C6.1, C7.1, C8.1, C9.1
- net ADC_ALRT: now also J21.2 (Pin_2); no longer U6.1 (P10)
- net GND: now also C1.2, C10.2, C11.2, C12.2, C13.2, C2.2, C5.2, C6.2, C7.2, C8.2, C9.2
- net SIM_DTR: now also J20.16 (Pin_16); no longer U6.20 (P07)
- net ~SIM_EN: now also J20.12 (Pin_12); no longer U6.19 (P06)
- net P00: now reaches U6.13 (P00)
- net P00: now also J20.1 (Pin_1)
- net P01: now reaches U6.14 (P01)
- net P01: now also J20.3 (Pin_3)
- net P02: now reaches U6.15 (P02)
- net P02: now also J20.5 (Pin_5)
- net P03: now reaches U6.16 (P03)
- net P03: now also J20.7 (Pin_7)
- net P04: now reaches U6.17 (P04)
- net P04: now also J20.9 (Pin_9)
- net P05: now reaches U6.18 (P05)
- net P05: now also J20.11 (Pin_11)
- net P11: now reaches U6.2 (P11)
- net P11: now also J21.3 (Pin_3)
- net P12: now reaches U6.3 (P12)
- net P12: now also J21.5 (Pin_5)
- net P13: now reaches U6.4 (P13)
- net P13: now also J21.7 (Pin_7)
- net P14: now reaches U6.5 (P14)
- net P14: now also J21.9 (Pin_9)
- net P15: now reaches U6.6 (P15)
- net P15: now also J21.11 (Pin_11)
- net P16: now reaches U6.7 (P16)
- net P16: now also J21.13 (Pin_13)
- net P17: now reaches U6.8 (P17)
- net P17: now also J21.15 (Pin_15)
- new net P06: J20.13 (Pin_13), U6.19 (P06)
- new net P07: J20.15 (Pin_15), U6.20 (P07)
- new net P10: J21.1 (Pin_1), U6.1 (P10)
- new net SIM_RST: J20.14 (Pin_14)
- no-connect marks 177 -> 186
Other:
- sheet SIM800L ports: added RST; removed none
- note added: "Buffer Caps"
- note added: "TTL Adapter / Chip needed (not worth it)"

Commit message: PCB Fixes
Parts:
- added C14: 10u, symbol Device:C
Connections:
- net GND: now also C14.2
- net at J1.2 (Pin_2), J9.1 (Pin_1), U4.1 (VDD): now also C14.1
Other:
- note added: "Buffer Capacitor, sonst Flicker"
Changed lines of the file:
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@@
 	(generator_version "9.0")
 	(paper "A4")
+	(text "Buffer Capacitor, sonst Flicker"
+		(exclude_from_sim no)
+		(at 96.774 20.828 0)
+		(effects
+			(font
+				(size 0.762 0.762)
+			)
+		)
+	)
 	(text "TTL Adapter / \nChip needed\n(not worth it)"
 		(exclude_from_sim no)
@@
 	)
 	(junction
+		(at 68.58 48.26)
+		(diameter 0)
+		(color 0 0 0 0)
+	)
+	(junction
 		(at 72.39 73.66)
 		(diameter 0)
@@
 	(wire
 		(pts
+			(xy 62.23 48.26) (xy 68.58 48.26)
+		)
+		(stroke
+			(width 0)
+			(type default)
+		)
+	)
+	(wire
+		(pts
 			(xy 81.28 24.13) (xy 95.25 24.13)
 		)
@@
 	(wire
 		(pts
+			(xy 62.23 44.45) (xy 62.23 48.26)
+		)
+		(stroke
+			(width 0)
+			(type default)
+		)
+	)
+	(wire
+		(pts
 			(xy 66.04 88.9) (xy 71.12 88.9)
 		)
@@
 	(wire
 		(pts
+			(xy 62.23 36.83) (xy 62.23 34.29)
+		)
+		(stroke
+			(width 0)
+			(type default)
+		)
+	)
+	(wire
+		(pts
 			(xy 267.97 78.74) (xy 267.97 82.55)
 		)
@@
 					(unit 1)
 				)
+			)
+		)
+	)
+	(symbol
+		(lib_id "Device:C")
+		(at 62.23 40.64 0)
+		(unit 1)
+		(exclude_from_sim no)
+		(in_bom yes)
+		(on_board yes)
+		(dnp no)
+		(fields_autoplaced yes)
+		(property "Reference" "C14"
+			(at 66.04 39.3699 0)
+			(effects
+				(font
+					(size 1.27 1.27)
+				)
+				(justify left)
+			)
+		)
+		(property "Value" "10u"
+			(at 66.04 41.9099 0)
+			(effects
+				(font
+					(size 1.27 1.27)
+				)
+				(justify left)
+			)
+		)
+		(property "Footprint" ""
+			(at 63.1952 44.45 0)
+			(effects
+				(font
+					(size 1.27 1.27)
+				)
+				(hide yes)
+			)
+		)
+		(property "Datasheet" "~"
+			(at 62.23 40.64 0)
+			(effects
+				(font
+					(size 1.27 1.27)
+				)
+				(hide yes)
+			)
+		)
+		(property "Description" "Unpolarized capacitor"
+			(at 62.23 40.64 0)
+			(effects
+				(font
+					(size 1.27 1.27)
+				)
+				(hide yes)
+			)
+		)
+		(pin "1"
+		)
+		(pin "2"
+		)
+		(instances
+			(project ""
+				(path "/88bb7a71-704b-4bd6-bab4-d44bdefe0db1"
+					(reference "C14")
+					(unit 1)
+				)
