File: KiCad Files/Bojen_PCB/SIM800L.kicad_sch (KiCad schematic)
At the start: 4 parts, among them Q1 IRF5210PBF, U3 SIM800L-CORE

Commit message: tft Screen QR Code Display
Other:
- note added: "RST Pin auf GPIO TODO"
Changed lines of the file:
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@@
 	(generator_version "9.0")
 	(paper "A4")
+	(text "RST Pin auf GPIO TODO"
+		(exclude_from_sim no)
+		(at 81.534 99.822 0)
+		(effects
+			(font
+				(size 1.27 1.27)
+			)
+		)
+	)
 	(text "Gate Resistor limits max inrush current \non gpio from Gate Capacitance."
 		(exclude_from_sim no)

Commit message: PCB Updated, Fixes
Parts:
- added C3: 100u, Capacitor_THT:CP_Radial_D8.0mm_P5.00mm, symbol Device:C_Polarized
- added C4: 10u, Capacitor_THT:C_Axial_L5.1mm_D3.1mm_P10.00mm_Horizontal, symbol Device:C
- added J29: Sim PWR Skip, Connector_PinHeader_2.54mm:PinHeader_1x02_P2.54mm_Vertical, symbol Connector_Generic:Conn_01x02
Connections:
- net GND: now also C3.2, C4.2
- net Vin: now also J29.1 (Pin_1)
- net at Q1.2 (D), U3.2 (VCC): now also C3.1, C4.1, J29.2 (Pin_2)
- net RST: now reaches U3.3 (RST)
- no-connect marks 7 -> 6
Other:
- note added: "Buffer Caps"
- moved on the sheet: Q1, R1, R2

Commit message: PCB Fixes
Parts:
- added Q2: NPN, symbol Simulation_SPICE:NPN
- added R7: 10K, symbol Device:R
Connections:
- net GND: now also Q2.3 (E)
- net ~EN: now also R7.1; no longer R2.1
- new net: Q2.1 (C), R2.1
- new net: Q2.2 (B), R7.2
Other:
- note added: "DOES NOT WORK, Wenn ESP aus, wird gpio auf GND gezogen, ~1.1V gemessen Spannungsteiler innenwiderstand berechnen? Auf Nicht inv. wechseln"
