File: KiCad Files/Bojen_PCB/Version2/ESP32.kicad_sch (KiCad schematic)
At the start: 3 parts, among them J3 GPIO Breakout 2, J8 GPIO Breakout 1, U7 ESP32-DEVKIT-V1

Commit message: state_module, Bilder
Other:
- company: (none) -> Alexander Mohr
- title: (none) -> Datenbojen
Changed lines of the file:
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@@
 	(generator_version "9.0")
 	(paper "A4")
+	(title_block
+		(title "Datenbojen")
+		(rev "2")
+		(company "Alexander Mohr")
+		(comment 1 "TU Berlin")
+	)
 	(text "Jumper Connection to\n Readjust Pinout"
 		(exclude_from_sim no)
