File: KiCad Files/Bojen_PCB/Version2/SIM800L.kicad_sch (KiCad schematic)
At the start: 4 parts, among them Q1 IRF5210PBF, U3 SIM800L-CORE

Commit message: state_module, Bilder
Other:
- company: (none) -> Alexander Mohr
- title: (none) -> Datenbojen
Changed lines of the file:
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@@
 	(generator_version "9.0")
 	(paper "A4")
+	(title_block
+		(title "Datenbojen")
+		(rev "2")
+		(company "Alexander Mohr")
+		(comment 1 "TU Berlin")
+	)
 	(text "Gate Resistor limits max inrush current \non gpio from Gate Capacitance."
 		(exclude_from_sim no)
