File: KiCad Files/Bojen_PCB/Version2/sensors.kicad_sch (KiCad schematic)
At the start: 14 parts, among them J20 TMP PUL UP, J21 TMP PULL DOWN, J22 TMP Sens, J24 TDS Sens, J25 PH Sens, J26 DO Sens, J27 TRB Sens, U11 DO Sensor, U15 PH Sensor, U5 ADC - ADS1115 Module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

Commit message: state_module, Bilder
Other:
- company: (none) -> Alexander Mohr
- title: (none) -> Datenbojen
Changed lines of the file:
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@@
 	(generator_version "9.0")
 	(paper "A4")
+	(title_block
+		(title "Datenbojen")
+		(rev "2")
+		(company "Alexander Mohr")
+		(comment 1 "TU Berlin")
+	)
 	(junction
 		(at 189.23 95.25)
